File: pcb/eyocean_carrier.kicad_pcb (KiCad board)
At the start: 2 copper layers, 56 x 32 mm, 9 parts, among them J1 SuperMini_L (TX..GPIO7), J2 SuperMini_R (5V..GPIO8), J3 CC1101_433MHz

Commit message: pcb: use 0603 for both decoupling capacitors
Move the 10 uF CC1101 decoupling cap from 0805 to the same 0603
hand-solder footprint as the 100 nF (use X5R, >= 6.3 V). Regenerated
schematic and board (3V3 rail and pad-1 positions unchanged), ERC/DRC
with schematic parity clean, JLCPCB Gerbers re-exported.
Parts:
- C2: footprint Capacitor_SMD:C_0805_2012Metric_Pad1.18x1.45mm_HandSolder -> Capacitor_SMD:C_0603_1608Metric_Pad1.08x0.95mm_HandSolder
- moved C2 0.18 mm to (133.3, 108.8)

Commit message: pcb: single 10 uF decoupling capacitor
The CC1101 module already carries its own 100 nF next to the chip, so
the carrier only needs a local bulk cap for the TX current bursts. Drop
C2 and make C1 a 10 uF 0603 X5R 10 V (LCSC C19702, Samsung
CL10A106KP8NNNC); its GND stitching via now sits beside its pad.
Regenerated schematic and board, ERC/DRC with schematic parity clean,
JLCPCB Gerbers re-exported.
Parts:
- removed C2: 10uF, Capacitor_SMD:C_0603_1608Metric_Pad1.08x0.95mm_HandSolder
- C1: value 100nF -> 10uF

Commit message: feat: direct-solder stack-up, centred CC1101 header, cad build guide
Both modules are now soldered straight onto the carrier through their
male headers (no sockets), so the case is recomputed from a direct-solder
stack-up: separate SuperMini / CC1101 header-spacer heights, SMA axis
offset, pin-tail room. Case 60.5 x 37 x 18.1 mm (was 26.6 mm tall).

- M2 x 16 flat-head bolts sit flush; the hex nut pocket depth is now
  automatic so the head stays flush when measured spacers shift the
  roof, and base standoffs are 6.5 mm for a printable nut wall.
- Fit checks refuse to export when the bolt, pin tails, SMA/carrier
  clearance or nut wall don't fit.
- Carrier shortened to 53.5 mm so the CC1101 SMA barrel overhangs the
  board edge instead of hitting it at the lower height.
- CC1101 header rows are centred on the module's 15 mm edge (measured
  from both CC1101_specs drawings; the table's F = 1.5 was wrong). Pads
  and routing are unchanged; the module outline and the SMA hole move.
- New cad/README.md build guide (prerequisites, height stack-up with
  formulas, what to measure, export, print, hardware, assembly,
  troubleshooting). README parts list and assembly updated.
- Regenerated schematic/board (ERC/DRC/parity clean), JLCPCB Gerbers,
  STL/3MF parts and render.
Parts:
- moved H2 2.50 mm to (150.5, 103.0)
- moved H4 2.50 mm to (150.5, 129.0)
Other:
- board size 56 x 32 mm -> 53.5 x 32 mm

Commit message: pcb: move 10 uF decoupling cap to the back, 3V3 on B.Cu
C1 now sits on B.Cu under its old spot, clear of the CC1101 module and
easy to solder after both modules are fitted; the case leaves 3.5 mm
under the board (cap <= 0.95 mm tall). +3V3 is routed on B.Cu at 0.6 mm
along the north margin to C1 and on to CC1101 VDD.

The change was made in the KiCad GUI and is ported into gen_pcb.py
(flip_to_back + new 3V3 route) so build.sh reproduces it; the
regenerated board matches the GUI edit segment-for-segment. ERC/DRC
with schematic parity clean; JLCPCB Gerbers re-exported. Assembly
notes in README.md and cad/README.md updated.
Parts:
- C1: moved to B.Cu
Routing:
- net +3V3: track 36.1 -> 33.5 mm
